File: 03010 - xMM2/cad/03010-002/03010-002.kicad_sch (KiCad schematic)
At the start: 46 parts, among them J1 Conn_01x04_Pin, Q1 2N7000, Q2 2N7000, Q3 2N7000, Q4 2N7000, SW1 SW_Reed, SW10 SW_Reed, SW11 SW_Reed, SW12 SW_Reed, SW13 SW_Reed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

Commit message: updated 03010-002
Parts:
- added JP1: Jumper_2_Bridged, Connector_PinHeader_2.54mm:PinHeader_1x02_P2.54mm_Vertical, symbol Jumper:Jumper_2_Bridged
- BZ1: footprint (none) -> Buzzer_Beeper:Buzzer_12x9.5RM7.6
- C1: footprint (none) -> Capacitor_THT:C_Disc_D5.1mm_W3.2mm_P5.00mm
- D2: renamed from D1; footprint (none) -> LED_THT:LED_D5.0mm-4_RGB
- D3: renamed from D2; footprint (none) -> LED_THT:LED_D5.0mm-4_RGB
- D4: renamed from D3; footprint (none) -> LED_THT:LED_D5.0mm-4_RGB
- D5: renamed from D4; footprint (none) -> LED_THT:LED_D5.0mm-4_RGB
- J1: footprint (none) -> Connector_JST:JST_XH_B4B-XH-A_1x04_P2.50mm_Vertical
- R1, R10, R11, R12, R13, R14, R15, R16, R17, R18, R2, R3, R4, R5, R6, R7, R8, R9: footprint (none) -> Resistor_THT:R_Axial_DIN0207_L6.3mm_D2.5mm_P10.16mm_Horizontal
- SW1, SW10, SW11, SW12, SW13, SW14, SW2, SW3, SW4, SW5, SW6, SW7, SW8, SW9: footprint (none) -> custom_footprints:MS_REED_SWITCH
- USB-C1: renamed from USB-C; footprint (none) -> Connector_JST:JST_XH_B4B-XH-A_1x04_P2.50mm_Vertical
Connections:
- net at U1.15 (PB1): now also JP1.1 (A); no longer R15.2
- new net: JP1.2 (B), R15.2
Other:
- moved on the sheet: BZ1, D1, D2, D3, D4, D5, Q1, Q2, Q3, Q4, R15, R16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
