File: 22001 - RP2040 AVR PROG/cad/22001.kicad_pcb (KiCad board)
At the start: 2 copper layers, 79 x 52.8 mm, 8 parts, among them J2 Conn_01x14_Pin, J3 Conn_01x14_Pin, J4 Conn_01x14_Pin, J5 Conn_01x14_Pin, U1 ATmega328-P

Commit message: updated pcb design
Other:
- board text added: "SN: QC:"
Changed lines of the file:
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@@
 		(tenting front back)
 		(pcbplotparams
-			(layerselection 0x00000000_00000000_55555555_57555551)
-			(plot_on_all_layers_selection 0x00000000_00000000_00000000_00000000)
+			(layerselection 0x00000000_00000000_55555555_55555570)
+			(plot_on_all_layers_selection 0x00000000_00000000_00000000_02000000)
 			(disableapertmacros no)
 			(usegerberextensions no)
@@
 		(layer "Edge.Cuts")
 	)
+	(gr_text "SN:\nQC:"
+		(at 150 30.75 0)
+		(layer "F.SilkS")
+		(effects
+			(font
+				(size 1.8 1.8)
+				(thickness 0.4)
+				(bold yes)
+			)
+			(justify left bottom)
+		)
+	)
 	(gr_text "MARIAN SCIENTIFIC"
-		(at 97.52 32.16 0)
+		(at 97.75 29.25 0)
 		(layer "F.SilkS")
 		(effects
@@
 	)
 	(gr_text "22001\nRP2040-ZERO\nATMEGA328\nPROGRAMMER\n\nARTISANALLY\nCRAFTED IN\nBRIDGEPORT, CT"
-		(at 154.45 64.09 0)
+		(at 155 63.75 0)
 		(layer "F.SilkS")
 		(effects
 			(font
-				(size 1.5 1.5)
-				(thickness 0.2)
+				(size 1.8 1.8)
+				(thickness 0.4)
+				(bold yes)
 			)
 		)
