File: 02004 - FireWireUSBCPD/CAD/02004-001/FireWireUSBCPD/02004-001.kicad_pcb (KiCad board)
At the start: 2 copper layers, 55.5 x 37.5 mm, 12 parts, among them J1 IEEE1394a, P1 USB_C_Plug_USB2.0, U1 CH224K

Commit message: Add files via upload
Parts:
- moved C4 5.52 mm to (90.5, 35.0)
Routing:
- net GND: track 99.1 -> 111.1 mm
- net Net-(D1-A): track 137.0 -> 148.7 mm
- net Net-(P1-CC): track 16.1 -> 25.0 mm
- net unconnected-(P1-VCONN-PadB5): track 0.00 -> 2.12 mm
Other:
- outline, holes or cut-outs redrawn
- board text added: "Anthony 02004-001"
- board text removed: "02004-001 Anthony"

Commit message: Add files via upload
Routing:
- net Net-(U1-CFG1): track 10.4 -> 9.85 mm
Other:
- board text added: "02004-001 FEB 8, 2026 REV3 AF"
- board text removed: "Anthony 02004-001"
Changed lines of the file:
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@@
 	)
 	(gr_rect
-		(start 85.5 45)
+		(start 85.5 46)
 		(end 91.5 53)
 		(stroke
@@
 	)
 	(gr_rect
-		(start 93 49)
+		(start 93 50)
 		(end 100.9 56.5)
 		(stroke
@@
 		(layer "Edge.Cuts")
 	)
-	(gr_text "Anthony\n02004-001\n"
-		(at 65.5 36 0)
+	(gr_text "02004-001\nFEB 8, 2026\nREV3 AF\n\n"
+		(at 69.5 40 0)
 		(layer "B.SilkS")
 		(effects
@@
 		(start 77.225 38)
 		(end 75 38)
-		(width 0.8)
+		(width 0.6)
 		(layer "F.Cu")
 		(net 3)
@@
 		(start 84 41.5)
 		(end 84.5 42)
-		(width 0.8)
+		(width 0.6)
 		(layer "F.Cu")
 		(net 13)
@@
 		(start 83.5 41)
 		(end 84 41.5)
-		(width 0.8)
+		(width 0.6)
 		(layer "F.Cu")
 		(net 13)
@@
 		(start 82.5 42)
 		(end 82.5 44)
-		(width 0.8)
+		(width 0.6)
 		(layer "F.Cu")
 		(net 13)
@@
 		(start 82.5 41)
 		(end 83.5 41)
-		(width 0.8)
+		(width 0.6)
 		(layer "F.Cu")
 		(net 13)
 	)
 	(segment
-		(start 85 35.5)
-		(end 85 39)
-		(width 0.6)
-		(layer "F.Cu")
-		(net 14)
-	)
-	(segment
-		(start 85 39)
+		(start 84 39)
 		(end 82.5 39)
 		(width 0.6)
@@
 	)
 	(segment
+		(start 85 35.5)
+		(end 85 38)
+		(width 0.6)
+		(layer "F.Cu")
+		(net 14)
+	)
+	(segment
 		(start 83.95 34.45)
 		(end 85 35.5)
@@
 		(layer "F.Cu")
 		(net 14)
+	)
+	(segment
+		(start 85 38)
+		(end 84 39)
+		(width 0.6)
+		(layer "F.Cu")
+		(net 14)

Commit message: Add files via upload
Parts:
- moved R4 2.00 mm to (88.5, 54.5)
Routing:
- net Net-(D1-A): track 148.7 -> 143.8 mm
- net GND: track 111.1 -> 114.8 mm
Other:
- board text added: "02004-001 FEB 10, 2026 REV4 AF"
- board text removed: "02004-001 FEB 8, 2026 REV3 AF"
Changed lines of the file:
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@@
 	(footprint "Resistor_SMD:R_1206_3216Metric_Pad1.30x1.75mm_HandSolder"
 		(layer "F.Cu")
-		(at 90.5 54.5 -90)
+		(at 88.5 54.5 -90)
 		(descr "Resistor SMD 1206 (3216 Metric), square (rectangular) end terminal, IPC-7351 nominal with elongated pad for handsoldering. (Body size source: IPC-SM-782 page 72, https://www.pcb-3d.com/wordpress/wp-content/uploads/ipc-sm-782a_amendment_1_and_2.pdf), generated with kicad-footprint-generator")
 		(tags "resistor handsolder")
@@
 	(gr_rect
 		(start 85.5 46)
-		(end 91.5 53)
+		(end 91.1 53)
 		(stroke
 			(width 0.2)
@@
 		(net 2)
 	)
+	(gr_line
+		(start 92.5 49.5)
+		(end 92.5 51.1)
+		(stroke
+			(width 0.6)
+			(type solid)
+		)
+		(layer "F.Cu")
+		(net 1)
+	)
 	(gr_rect
 		(start 71 25.3)
@@
 	(gr_rect
 		(start 86 38.25)
-		(end 91.5 40.25)
+		(end 91 40.25)
 		(stroke
 			(width 0.2)
@@
 	)
 	(gr_rect
-		(start 93 50)
+		(start 92.3 50)
 		(end 100.9 56.5)
 		(stroke
@@
 		(layer "Edge.Cuts")
 	)
-	(gr_text "02004-001\nFEB 8, 2026\nREV3 AF\n\n"
+	(gr_text "02004-001\nFEB 10, 2026\nREV4 AF\n\n"
 		(at 69.5 40 0)
 		(layer "B.SilkS")
@@
 	)
 	(segment
-		(start 94.48 45.02)
-		(end 95.62 45.02)
-		(width 0.8)
-		(layer "F.Cu")
-		(net 1)
-	)
-	(segment
 		(start 72.5 56.05)
 		(end 90.5 56.05)
@@
 	)
 	(segment
-		(start 93.5 38.5)
-		(end 91.5625 36.5625)
-		(width 0.8)
-		(layer "F.Cu")
-		(net 1)
-	)
-	(segment
 		(start 72.5 58.5)
 		(end 72 59)
@@
 	)
 	(segment
-		(start 93.5 46)
-		(end 94.48 45.02)
-		(width 0.8)
-		(layer "F.Cu")
-		(net 1)
-	)
-	(segment
 		(start 50 59)
 		(end 50 35)
@@
 	)
 	(segment
+		(start 92 37)
+		(end 91.5625 36.5625)
+		(width 0.8)
+		(layer "F.Cu")
+		(net 1)
+	)
+	(segment
 		(start 96.98 41.98)
 		(end 95.62 41.98)
@@
 	)
 	(segment
+		(start 95.6 45)
+		(end 95.62 45.02)
+		(width 0.8)
+		(layer "F.Cu")
+		(net 1)
+	)
+	(segment
+		(start 92.45 56.05)
+		(end 93.5 55)
+		(width 0.8)
+		(layer "F.Cu")
+		(net 1)
+	)
+	(segment
+		(start 68.5 42)
+		(end 67.5 41)
+		(width 0.8)
+		(layer "F.Cu")
+		(net 1)
+	)
+	(segment
+		(start 90.5 56.05)
+		(end 92.45 56.05)
+		(width 0.8)
+		(layer "F.Cu")
+		(net 1)
+	)
+	(segment
+		(start 59.5 41)
+		(end 59.5 41.55)
+		(width 0.8)
+		(layer "F.Cu")
+		(net 1)
+	)
+	(segment
+		(start 72.45 56)
+		(end 72.5 56.05)
+		(width 0.8)
+		(layer "F.Cu")
+		(net 1)
+	)
+	(segment
+		(start 97 42)
+		(end 96.98 41.98)
+		(width 0.8)
+		(layer "F.Cu")
+		(net 1)
+	)
+	(segment
+		(start 93.98 45.02)
+		(end 95.62 45.02)
+		(width 0.6)
+		(layer "F.Cu")
+		(net 1)
+	)
+	(segment
+		(start 92 39.96)
+		(end 92 37)
+		(width 0.6)
+		(layer "F.Cu")
+		(net 1)
+	)
+	(segment
+		(start 95.62 45.02)
+		(end 97.98 45.02)
+		(width 0.8)
+		(layer "F.Cu")
+		(net 1)
+	)
+	(segment
+		(start 59.5 41.55)
+		(end 59.05 42)
+		(width 0.8)
+		(layer "F.Cu")
+		(net 1)
+	)
+	(segment
+		(start 68.4375 31.5)
+		(end 68.4375 41.9375)
+		(width 0.8)
+		(layer "F.Cu")
+		(net 1)
+	)
+	(segment
+		(start 92.5 46.5)
+		(end 93.98 45.02)
+		(width 0.6)
+		(layer "F.Cu")
+		(net 1)
+	)
+	(segment
+		(start 53.5 31.5)
+		(end 68.4375 31.5)
+		(width 0.8)
+		(layer "F.Cu")
+		(net 1)
+	)
+	(segment
+		(start 98 42)
+		(end 97 42)
+		(width 0.8)
+		(layer "F.Cu")
+		(net 1)
+	)
+	(segment
+		(start 97.98 45.02)
+		(end 98 45)
+		(width 0.8)
+		(layer "F.Cu")
+		(net 1)
+	)
+	(segment
+		(start 50 35)
+		(end 53.5 31.5)
+		(width 0.8)
+		(layer "F.Cu")
+		(net 1)
+	)
+	(segment
+		(start 94.02 41.98)
+		(end 92 39.96)
+		(width 0.6)
+		(layer "F.Cu")
+		(net 1)
+	)
+	(segment
+		(start 72.5 56.05)
+		(end 72.5 58.5)
+		(width 0.8)
+		(layer "F.Cu")
+		(net 1)
+	)
+	(segment
+		(start 68.4375 41.9375)
+		(end 68.5 42)
+		(width 0.8)
+		(layer "F.Cu")
+		(net 1)
+	)
+	(segment
+		(start 95.62 41.98)
+		(end 94.02 41.98)
+		(width 0.6)
+		(layer "F.Cu")
+		(net 1)
+	)
+	(segment
 		(start 91.5625 36.5625)
 		(end 90.5 36.5625)
@@
 	)
 	(segment
-		(start 95.6 45)
-		(end 95.62 45.02)
-		(width 0.8)
-		(layer "F.Cu")
-		(net 1)
-	)
-	(segment
-		(start 92.45 56.05)
-		(end 93.5 55)
-		(width 0.8)
-		(layer "F.Cu")
-		(net 1)
-	)
-	(segment
-		(start 95.5375 42.0625)
-		(end 95.62 41.98)
-		(width 0.8)
-		(layer "F.Cu")
-		(net 1)
-	)
-	(segment
-		(start 68.5 42)
-		(end 67.5 41)
-		(width 0.8)
-		(layer "F.Cu")
-		(net 1)
-	)
-	(segment
-		(start 93.5 41.46)
-		(end 93.5 38.5)
-		(width 0.8)
-		(layer "F.Cu")
-		(net 1)
-	)
-	(segment
-		(start 90.5 56.05)
-		(end 92.45 56.05)
-		(width 0.8)
-		(layer "F.Cu")
-		(net 1)
-	)
-	(segment
-		(start 59.5 41)
-		(end 59.5 41.55)
-		(width 0.8)
-		(layer "F.Cu")
-		(net 1)
-	)
-	(segment
-		(start 72.45 56)
-		(end 72.5 56.05)
-		(width 0.8)
-		(layer "F.Cu")
-		(net 1)
-	)
-	(segment
-		(start 97 42)
-		(end 96.98 41.98)
-		(width 0.8)
-		(layer "F.Cu")
-		(net 1)
-	)
-	(segment
-		(start 95.62 45.02)
-		(end 97.98 45.02)
-		(width 0.8)
-		(layer "F.Cu")
-		(net 1)
-	)
-	(segment
-		(start 59.5 41.55)
-		(end 59.05 42)
-		(width 0.8)
-		(layer "F.Cu")
-		(net 1)
-	)
-	(segment
-		(start 68.4375 31.5)
-		(end 68.4375 41.9375)
-		(width 0.8)
-		(layer "F.Cu")
-		(net 1)
-	)
-	(segment
-		(start 94.02 41.98)
-		(end 94 42)
-		(width 0.8)
-		(layer "F.Cu")
-		(net 1)
-	)
-	(segment
-		(start 53.5 31.5)
-		(end 68.4375 31.5)
-		(width 0.8)
-		(layer "F.Cu")
-		(net 1)
-	)
-	(segment
-		(start 98 42)
-		(end 97 42)
-		(width 0.8)
-		(layer "F.Cu")
-		(net 1)
-	)
-	(segment
-		(start 97.98 45.02)
-		(end 98 45)
-		(width 0.8)
-		(layer "F.Cu")
-		(net 1)
-	)
-	(segment
-		(start 50 35)
-		(end 53.5 31.5)
-		(width 0.8)
-		(layer "F.Cu")
-		(net 1)
-	)
-	(segment
-		(start 72.5 56.05)
-		(end 72.5 58.5)
-		(width 0.8)
-		(layer "F.Cu")
-		(net 1)
-	)
-	(segment
-		(start 93.5 55)
-		(end 93.5 46)
-		(width 0.8)
-		(layer "F.Cu")
-		(net 1)
-	)
-	(segment
-		(start 68.4375 41.9375)
-		(end 68.5 42)
-		(width 0.8)
-		(layer "F.Cu")
-		(net 1)
-	)
-	(segment
-		(start 95.62 41.98)
-		(end 94.02 41.98)
-		(width 0.8)
-		(layer "F.Cu")
-		(net 1)
-	)
-	(segment
-		(start 94.02 41.98)
-		(end 93.5 41.46)
-		(width 0.8)
+		(start 92.5 49.5)
+		(end 92.5 46.5)
+		(width 0.6)
 		(layer "F.Cu")
 		(net 1)
@@
 	)
 	(segment
+		(start 94.15 46.25)
+		(end 93.9 46.5)
+		(width 0.8)
+		(layer "F.Cu")
+		(net 2)
+	)
+	(segment
 		(start 97.5 40.75)
 		(end 97.5 32)
@@
 	)
 	(segment
+		(start 95.62 40.75)
+		(end 94.25 40.75)
+		(width 0.8)
+		(layer "F.Cu")
+		(net 2)
+	)
+	(segment
+		(start 94.25 40.75)
+		(end 93.9 40.4)
+		(width 0.8)
+		(layer "F.Cu")
+		(net 2)
+	)
+	(segment
 		(start 82.5625 50.5625)
 		(end 79.8625 47.8625)
@@
 		(width 0.8)
 		(layer "F.Cu")
+		(net 2)
+	)
+	(segment
+		(start 95.62 46.25)
+		(end 94.15 46.25)
+		(width 0.8)
+		(layer "F.Cu")
