File: 02004 - FireWireUSBCPD/CAD/02004-004/02004-004.kicad_pcb (KiCad board)
At the start: 2 copper layers, 48 x 29 mm, 11 parts, among them J1 IEEE1394a, P1 USB_C_Plug_USB2.0, U1 CH224K

Commit message: 02004-004 fab files and 004T1
Parts:
- added REF**: MountingHole_3.2mm_M3, MountingHole:MountingHole_3.2mm_M3, F.Cu at (89.5, 54.8)
- added REF**: MountingHole_3.2mm_M3, MountingHole:MountingHole_3.2mm_M3, F.Cu at (49.5, 33.2)
- added REF**: MountingHole_3.2mm_M3, MountingHole:MountingHole_3.2mm_M3, F.Cu at (89.5, 33.2)
- added REF**: MountingHole_3.2mm_M3, MountingHole:MountingHole_3.2mm_M3, F.Cu at (49.5, 54.8)
Other:
- outline, holes or cut-outs redrawn
