File: 03007 - Axial Flux Stepper Motor/resources/circuit/03007-007/03007-007.kicad_pcb (KiCad board)
At the start: 2 copper layers, 87 x 50 mm, 49 parts, among them J1 USB_C_Receptacle_USB2.0_14P, J2 Screw_Terminal_01x02, J3 Screw_Terminal_01x02, J4 Screw_Terminal_01x02, J5 Screw_Terminal_01x02, J6 Screw_Terminal_01x02, J7 Conn_01x04_Pin, U1 SN754410NE, U2 SN754410NE, U3 CH32V003AxMx

Commit message: 03007-007 pcb
Parts:
- moved D12 174.6 mm to (219.2, 95.2), turned to -90 degrees
- moved D1 170.2 mm to (225.8, 86.8), turned to -90 degrees
- moved D2 168.7 mm to (225.8, 95.2), turned to -90 degrees
- moved D3 168.1 mm to (219.2, 86.8), turned to -90 degrees
- moved D13 136.9 mm to (188.0, 103.5), turned to -90 degrees
- moved D11 136.6 mm to (190.8, 93.5), turned to -90 degrees
- moved D6 135.6 mm to (214.8, 101.4), turned to -90 degrees
- moved D14 135.0 mm to (188.0, 112.0), turned to -90 degrees
- moved R3 134.3 mm to (211.8, 98.3), turned to 90 degrees
- moved D7 131.8 mm to (208.8, 101.4), turned to 90 degrees
- moved J5 126.7 mm to (209.2, 73.5), turned to 180 degrees
- moved J4 124.9 mm to (195.0, 73.5), turned to 180 degrees
- moved D10 121.8 mm to (184.5, 93.5), turned to 90 degrees
- moved R5 121.6 mm to (187.5, 96.5), turned to -90 degrees
- moved C8 120.4 mm to (210.5, 89.5), turned to -90 degrees
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Connections:
- J1 pad S1: unconnected-(J1-SHIELD-PadS1) -> GND
- U1 pad 10: Net-(U1-2A) -> Net-(U1-3A)
- U1 pad 15: Net-(U1-1A) -> Net-(U1-4A)
- U2 pad 10: Net-(U2-2A) -> Net-(U2-3A)
- U2 pad 15: Net-(U2-1A) -> Net-(U2-4A)
- U3 pad 2: Net-(U2-2A) -> Net-(U2-3A)
- U3 pad 3: unconnected-(U3-PC3-Pad3) -> Net-(U2-2A)
- U3 pad 4: unconnected-(U3-PC4-Pad4) -> Net-(U2-4A)
- U3 pad 5: unconnected-(U3-PC6-Pad5) -> Net-(U1-2A)
- U3 pad 6: unconnected-(U3-PC7-Pad6) -> Net-(U1-1A)
- U3 pad 8: Net-(U1-1A) -> Net-(U1-4A)
- U3 pad 9: Net-(U1-2A) -> Net-(U1-3A)
Routing:
- net Net-(U2-2A): track 0.00 -> 132.7 mm, vias 0 -> 1
- net Net-(U2-1A): track 0.00 -> 119.7 mm
- net Net-(U2-4A): track 0.00 -> 112.8 mm, vias 0 -> 1
- net Net-(U2-3A): track 0.00 -> 106.2 mm
- net Net-(D1-A): track 0.00 -> 92.2 mm, vias 0 -> 1
- net Vdrive: track 94.1 -> 176.1 mm, vias 3 -> 6
- net Net-(J7-Pin_1): track 103.0 -> 173.1 mm, vias 5 -> 6
- net Net-(D12-K): track 0.00 -> 63.6 mm, vias 0 -> 1
- net Net-(D10-A): track 0.00 -> 61.5 mm, vias 0 -> 1
- net Net-(U1-2A): track 26.7 -> 86.0 mm, vias 0 -> 2
- net Net-(D13-A): track 0.00 -> 52.9 mm, vias 0 -> 2
- net GND: track 77.5 -> 115.6 mm, vias 0 -> 20
- net Net-(U1-1A): track 29.7 -> 60.3 mm, vias 0 -> 2
- net Net-(U1-4A): track 0.00 -> 22.1 mm
- net Net-(U1-3A): track 0.00 -> 19.1 mm
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- added copper zone on B.Cu, net GND
- added copper zone on F.Cu, net GND
- removed copper zone on B.Cu, net (none)
- removed copper zone on F.Cu, net (none)
Other:
- board size 87 x 50 mm -> 120 x 50 mm
- board text added: "BOARD: 120X50MM MOUNT: 109X39MM"
- board text added: "GND"
- board text added: "MARIAN SCIENTIFIC 03000-007 2026-03-02"
- board text added: "NRST"
- board text added: "SWDIO"
- board text added: "VDD"
- board text removed: "BOARD: 87X50MM MOUNT: 76X39MM"
- board text removed: "MARIAN SCIENTIFIC 03000-007 2026-03-01"
