File: 03007 - Axial Flux Stepper Motor/resources/circuit/03007-007/03007-007.kicad_sch (KiCad schematic)
At the start: 45 parts, among them J1 USB_C_Receptacle_USB2.0_14P, J2 Screw_Terminal_01x02, J3 Screw_Terminal_01x02, J4 Screw_Terminal_01x02, J5 Screw_Terminal_01x02, J6 Screw_Terminal_01x02, J7 Conn_01x04_Pin, U1 SN754410NE, U2 SN754410NE, U3 CH32V003AxMx

Commit message: 03007-007 pcb
Connections:
- net at U2.2 (1A), U3.1 (PC1): no longer U2.15 (4A)
- net at U2.10 (3A), U3.2 (PC2): no longer U2.7 (2A)
- net at U3.3 (PC3): now also U2.7 (2A)
- net at U3.4 (PC4): now also U2.15 (4A)
- net at U3.5 (PC6): now also U1.7 (2A)
- net at U3.6 (PC7): now also U1.2 (1A)
- net at U1.15 (4A), U3.8 (PD4): no longer U1.2 (1A)
- net at U1.10 (3A), U3.9 (PD5): no longer U1.7 (2A)
